File: attiny1614_accsupervisor.sch (KiCad schematic (older format))
At the start: 38 parts, among them J1 VXO7803-500-M-TR, J2 MSTBA_2,5_3-G, J3 Conn_01x02, J4 Conn_02x20_Odd_Even, J5 AVR-UPDI-6, K1 JSM1-12V-5, Q1 BC817, Q2 BC817, Q3 BC817, Q4 BSS84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

Commit message: Q4, Q5 PFETs pin swap fixed
P ch. MOSFETs drain-source swapped pins are now fixed
Connections:
- net 12V: now also Q4.2 (S); no longer Q4.3 (D)
- net ACC: now also Q5.2 (S); no longer Q5.3 (D)
- net at R6.1, R8.2: now also Q4.3 (D); no longer Q4.2 (S)
- net at R7.1, R9.2: now also Q5.3 (D); no longer Q5.2 (S)
Other:
- note added: "r02 note: Q4, Q5 pin 2, 3 net changed"
Changed lines of the file:
@@
 Sheet 1 1
 Title "ATTINY-ACC-Supervisor"
-Date "2020-09-01"
-Rev "r01"
+Date "2020-09-22"
+Rev "r02"
 Comp ""
 Comment1 ""
@@
 F 5 "BSS84-7-F" H 6350 3550 50  0001 C CNN "Manufacturer_Part_Number"
 	1    6350 3550
-	1    0    0    -1
+	1    0    0    1
 $EndComp
 $Comp
@@
 F 5 "BSS84-7-F" H 6350 5250 50  0001 C CNN "Manufacturer_Part_Number"
 	1    6350 5250
-	1    0    0    -1
+	1    0    0    1
 $EndComp
 $Comp
@@
 Connection ~ 1350 4000
 Connection ~ 3350 4000
+Text Notes 5400 3150 0    50   ~ 0
+r02 note: Q4, Q5 pin 2, 3 net changed
 $EndSCHEMATC

Commit message: UPDI_DATA/~RESET pullup added
10k pullup for UPDI_DATA/~RESET pin added
Parts:
- added R16: 10k, Resistor_SMD:R_1206_3216Metric_Pad1.42x1.75mm_HandSolder, symbol Device:R
Connections:
- net 3V3: now also R16.2
- net UPDI_DATA: now also R16.1
Other:
- note added: "r03 note: 10k pull-up for UPDI/~RESET"
Changed lines of the file:
@@
 Title "ATTINY-ACC-Supervisor"
 Date "2020-09-22"
-Rev "r02"
+Rev "r03"
 Comp ""
 Comment1 ""
@@
 3V3
 Wire Wire Line
-	10550 4300 10650 4300
+	10550 4300 10600 4300
 Text Label 10650 4300 0    50   ~ 0
 UPDI_DATA
@@
 Text Notes 5400 3150 0    50   ~ 0
 r02 note: Q4, Q5 pin 2, 3 net changed
+$Comp
+L Device:R R16
+U 1 1 5F6A2A3A
+P 10350 3950
+F 0 "R16" V 10143 3950 50  0000 C CNN
+F 1 "10k" V 10234 3950 50  0000 C CNN
+F 2 "Resistor_SMD:R_1206_3216Metric_Pad1.42x1.75mm_HandSolder" V 10280 3950 50  0001 C CNN
+F 3 "~" H 10350 3950 50  0001 C CNN
+F 4 "(Generic)" H 10350 3950 50  0001 C CNN "Manufacturer_Name"
+F 5 "(10k)" H 10350 3950 50  0001 C CNN "Manufacturer_Part_Number"
+	1    10350 3950
+	0    1    1    0
+$EndComp
+Wire Wire Line
+	10600 4300 10600 3950
+Connection ~ 10600 4300
+Wire Wire Line
+	10600 4300 10650 4300
+Wire Wire Line
+	10500 3950 10600 3950
+Wire Wire Line
+	10200 3950 10050 3950
+Connection ~ 10050 3950
+Text Notes 8700 3700 0    50   ~ 0
+r03 note: 10k pull-up for UPDI/~RESET
 $EndSCHEMATC
